File: vna_blocks/4371.kicad_block/4371.kicad_sch (KiCad schematic)
At the start: 30 parts, among them U16 LTC2122IUK-TRPBF

Commit message: hmc7044 design block
Parts:
- removed C145: 10u, Capacitor_SMD:C_0402_1005Metric, symbol Device:C_Small
- removed C147: 1u, Capacitor_SMD:C_0402_1005Metric, symbol Device:C_Small
- removed C149, C153, C159, C166, C167, C170, C173, C178, C179, C180, C181: 0.1u, Capacitor_SMD:C_0402_1005Metric, symbol Device:C_Small
- removed C151: 10p, Capacitor_SMD:C_0402_1005Metric, symbol Device:C_Small
- removed C172: 2.2u, Capacitor_SMD:C_0603_1608Metric, symbol Device:C_Small
- removed FB4: MPZ1608S601ATA00, Inductor_SMD:L_0603_1608Metric, symbol Device:FerriteBead_Small
- removed R63, R64, R76, R77: 200, Resistor_SMD:R_0402_1005Metric, symbol Device:R_Small_US
- removed R68, R79: 10, Resistor_SMD:R_0402_1005Metric, symbol Device:R_Small_US
- removed R69, R78: 100, Resistor_SMD:R_0402_1005Metric, symbol Device:R_Small_US
- removed R70, R71, R83, R84: 5, Resistor_SMD:R_0201_0603Metric, symbol Device:R_Small_US
- removed R85: 1k, Resistor_SMD:R_0402_1005Metric, symbol Device:R_Small_US
- removed U16: LTC2122IUK-TRPBF, VNA_fp:QFN-48_UK_LIT-L, symbol VNA_sym:LTC2122IUK-TRPBF
- added C23, C24, C40, C59: 1u, Capacitor_SMD:C_0402_1005Metric, symbol Device:C_Small
- added C25, C26, C28, C29, C30, C33, C34, C52, C53, C57, C58, C60, C61: 0.1u, Capacitor_SMD:C_0402_1005Metric, symbol Device:C_Small
- added C27, C31, C32, C35, C36, C37, C39, C47, C48, C49, C50, C51, C54: 10p, Capacitor_SMD:C_0402_1005Metric, symbol Device:C_Small
- added C38, C46: P21BNL300M5S, VNA_fp:P21BN, symbol Device:C_Small
- added C41: 10n, Capacitor_SMD:C_0201_0603Metric, symbol Device:C_Small
- added C42: 100n, Capacitor_SMD:C_0201_0603Metric, symbol Device:C_Small
- added U5: ADF4371BCCZ, VNA_fp:CC_48_4_ADI-L, symbol VNA_sym:ADF4371BCCZ
Connections:
- net GNDA: now also C23.2, C24.2, C25.2, C26.1, C27.2, C28.2, C29.2, C30.1, C31.2, C32.2, C33.1, C34.1, C35.2, C36.2, C37.1, C39.2, C40.2, C47.2, C48.2, C49.2, C50.2, C51.2, C52.2, C53.2, C54.2, C57.2, C58.2, C59.2, C60.2, C61.2, U5.1 (GND), U5.12 (GND), U5.13 (GND), U5.20 (GND), U5.24 (GND), U5.25 (GND), U5.28 (GND), U5.36 (GND), U5.37 (GND), U5.40 (TEST), U5.42 (GND), U5.48 (GND), U5.49 (EPAD), U5.9 (GND)
- new net: C41.2, U5.18 (RF8P)
- new net: C46.1, U5.26 (RF16P)
- new net: C38.2, U5.11 (RF32P)
- new net: C42.2, U5.22 (RFAUX8P)
- new net 3V3: C54.1, C57.1, U5.29 (VCC_MUX)
- new net 3V3_Synth: C26.2, C27.1, C28.1, C30.2, C31.1, C32.1, C33.2, C34.2, C35.1, C37.2, C40.1, C47.1, C48.1, C49.1, C50.1, C51.1, C52.1, C53.1, C58.1, C59.1, C60.1, C61.1, U5.14 (VCC_X4), U5.15 (VDD_X4), U5.16 (VCC_X1), U5.17 (VDD_X1), U5.21 (VCC_X2), U5.30 (VCC_3V), U5.31 (VDD_NDIV), U5.32 (VDD_LS), U5.38 (VCC_LDO_3V), U5.4 (VCC_CAL), U5.45 (VCC_REF), U5.46 (VDD_PFD), U5.47 (VDD_VP)
- new net 5V_Synth: C23.1, C24.1, C25.1, C29.1, C36.1, C39.1, U5.7 (VCC_VCO), U5.8 (VCC_LDO)
- new net CPOut: U5.2 (CPOUT)
- new net MUXOUT: U5.41 (MUXOUT)
- new net RF16: C46.2
- new net RF32: C38.1
- new net RF8: C41.1
- new net RF8_AUX: C42.1
- new net Ref_CLK_N: U5.44 (REFN)
- new net Ref_CLK_P: U5.43 (REFP)
- new net Synth_*CS: U5.33 (*CS)
- new net Synth_CE: U5.39 (CE)
- new net Synth_SCK: U5.35 (SCLK)
- new net Synth_SDIO: U5.34 (SDIO)
- new net VTune: U5.5 (VTUNE)
- no-connect marks 4 -> 2
Other:
- note added: "place close to pin 47"
