File: vna_blocks/5961.kicad_block/5961.kicad_sch (KiCad schematic)
At the start: 21 parts, among them U10 ADL5961ACCZ

Commit message: hmc7044 design block
Parts:
- removed C100, C102: 1n, Capacitor_SMD:C_0402_1005Metric, symbol Device:C_Small
- removed C101, C89: 4.7u, Capacitor_SMD:C_0603_1608Metric, symbol Device:C_Small
- removed C109, C86, C92, C99: P21BNL300M5S, Capacitor_SMD:C_0201_0603Metric, symbol Device:C_Small
- removed C110, C94, C95: 100n, Capacitor_SMD:C_0402_1005Metric, symbol Device:C_Small
- added C103, C117, C90, C96: P21BNL300M5S, Capacitor_SMD:C_0201_0603Metric, symbol Device:C_Small
- added C105, C87, C93: 4.7u, Capacitor_SMD:C_0603_1608Metric, symbol Device:C_Small
- added C106: 1n, Capacitor_SMD:C_0402_1005Metric, symbol Device:C_Small
- added C111, C112, C84: 0.1u, Capacitor_SMD:C_0402_1005Metric, symbol Device:C_Small
- added C116, C118: 100n, Capacitor_SMD:C_0402_1005Metric, symbol Device:C_Small
- C102: renamed from C98; footprint Capacitor_SMD:C_0402_1005Metric -> Capacitor_SMD:C_0201_0603Metric
- C108: value 100n -> 1n
- C83: value 4.7u -> 0.1u; footprint Capacitor_SMD:C_0603_1608Metric -> Capacitor_SMD:C_0402_1005Metric
Connections:
- net GNDA: now also C108.2, C105.1, C106.1, C116.1, C118.1, C87.2, C93.2; no longer C108.1, C83.2
- net at U10.1 (AVCC): now also C105.2, C106.2
- net at U10.10 (LOM): now also C103.2
- net at C104.1, U10.14 (OVCC): now also C108.1, C87.1, C93.1; no longer C83.1
- net at U10.15 (IFRP): now also C112.1
- net at U10.16 (IFRM): now also C111.1
- net at U10.17 (VCM): now also C116.2; no longer C108.2
- net at U10.19 (RFOUT): now also C117.1
- net at U10.22 (OVDD): now also C118.2
- net at U10.3 (RFIN): now also C90.2
- net at U10.6 (IFFM): now also C83.2
- net at U10.7 (IFFP): now also C84.2
- net at U10.9 (LOP): now also C96.2
- net at R31.2: now also C103.1
