File: vna_blocks/IF_Filters.kicad_block/IF_Filters.kicad_sch (KiCad schematic)
At the start: 7 parts

Commit message: hmc7044 design block
Parts:
- removed C118, C120: 10p, Capacitor_SMD:C_0402_1005Metric, symbol Device:C_Small
- removed R81, R82: 49.9, Resistor_SMD:R_0402_1005Metric, symbol Device:R_Small_US
- removed TP3, TP4: IF_TP, symbol Connector:TestPoint
- added C414: 27p, Capacitor_SMD:C_0402_1005Metric, symbol Device:C_Small
- added C415: 10p, Capacitor_SMD:C_0402_1005Metric, symbol Device:C_Small
- added R38, R39: 49.9, Resistor_SMD:R_0402_1005Metric, symbol Device:R_Small_US
- added TP10, TP6: IF_TP, VNA_fp:IF_TP, symbol Connector:TestPoint
- C119: value 27p -> 10p
Connections:
- net GNDA: now also C119.1, C415.2
- net at C119.2: now also C414.1, R38.2, TP6.1
- new net: C414.2, C415.1, R39.2, TP10.1
