File: vna_blocks/LNA.kicad_block/LNA.kicad_pcb (KiCad board)
At the start: 4 copper layers, 7 parts, among them U11 LT3041ADE-PBF

Commit message: hmc7044 design block
Parts:
- removed C131, C136: 10u, Capacitor_SMD:C_0402_1005Metric
- removed C134: 4.7u, Capacitor_SMD:C_0603_1608Metric
- removed R44: 49.9k, Resistor_SMD:R_0402_1005Metric
- removed R45: 140k, Resistor_SMD:R_0402_1005Metric
- removed R46: 10k, Resistor_SMD:R_0402_1005Metric
- removed U11: LT3041ADE-PBF, VNA_fp:05-08-1708_ADI-L
- added C63: 100n, Capacitor_SMD:C_0402_1005Metric, F.Cu at (-161.0, 163.6)
- added C64: 100n, Capacitor_SMD:C_0402_1005Metric, F.Cu at (-160.4, 168.2)
- added C65: 100n, Capacitor_SMD:C_0402_1005Metric, F.Cu at (-160.4, 162.0)
- added C68: 100n, Capacitor_SMD:C_0402_1005Metric, F.Cu at (-158.4, 162.0)
- added C69: 100n, Capacitor_SMD:C_0402_1005Metric, F.Cu at (-158.8, 168.4)
- added C70: 100n, Capacitor_SMD:C_0402_1005Metric, F.Cu at (-157.8, 168.4)
- added C73: 100n, Capacitor_SMD:C_0402_1005Metric, F.Cu at (-156.4, 168.0)
- added C74: P21BNL300M5S, VNA_fp:P21BN, F.Cu at (-152.2, 164.6)
- added C75: 10n, Capacitor_SMD:C_0402_1005Metric, F.Cu at (-147.0, 154.0)
- added C76: 1u, Capacitor_SMD:C_0402_1005Metric, F.Cu at (-146.0, 154.0)
- added Cp2: 1p, Capacitor_SMD:C_0402_1005Metric, F.Cu at (-148.0, 154.0)
- added IC5: LVA-273PN+, VNA_fp:DG1847_MNC-L, F.Cu at (-158.2, 165.0)
- added L3: BCR272JLC, VNA_fp:BCR-272, F.Cu at (-149.6, 158.6)

Commit message: new parts, design blocks updated
Parts:
- removed C63, C64, C65, C68, C69, C70, C73: 100n, Capacitor_SMD:C_0402_1005Metric
- removed C74: P21BNL300M5S, VNA_fp:P21BN
- removed C75: 10n, Capacitor_SMD:C_0402_1005Metric
- removed C76: 1u, Capacitor_SMD:C_0402_1005Metric
- removed Cp2: 1p, Capacitor_SMD:C_0402_1005Metric
- removed IC5: LVA-273PN+, VNA_fp:DG1847_MNC-L
- removed L3: BCR272JLC, VNA_fp:BCR-272
- added C283: 100n, Capacitor_SMD:C_0402_1005Metric, F.Cu at (126.8, 222.6)
- added C286: 100n, Capacitor_SMD:C_0402_1005Metric, F.Cu at (127.4, 227.2)
- added C288: 100n, Capacitor_SMD:C_0402_1005Metric, F.Cu at (127.4, 221.0)
- added C292: 100n, Capacitor_SMD:C_0402_1005Metric, F.Cu at (129.4, 221.0)
- added C293: 100n, Capacitor_SMD:C_0402_1005Metric, F.Cu at (129.0, 227.4)
- added C295: 100n, Capacitor_SMD:C_0402_1005Metric, F.Cu at (130.0, 227.4)
- added C297: 100n, Capacitor_SMD:C_0402_1005Metric, F.Cu at (131.4, 227.0)
- added C301: P21BNL300M5S, VNA_fp:P21BN, F.Cu at (135.6, 223.6)
- added C302: 10n, Capacitor_SMD:C_0402_1005Metric, F.Cu at (140.8, 213.0)
- added C304: 1u, Capacitor_SMD:C_0402_1005Metric, F.Cu at (141.8, 213.0)
- added Cp3: 1p, Capacitor_SMD:C_0402_1005Metric, F.Cu at (139.8, 213.0)
- added IC14: LVA-273PN+, VNA_fp:DG1847_MNC-L, F.Cu at (129.6, 224.0)
- added L7: BCR272JLC, VNA_fp:BCR-272, F.Cu at (137.9, 216.1)
